Commit message: tested and tuned both mpc and pd on the real env

File: assets/racer.urdf (robot description, URDF)
Before this commit: robot racer, 6 links, 5 joints
Links:
- link center_of_mass_link: mass 0 -> 0.000001
- link prop0_link: mass 0 -> 0.000001
- link prop1_link: mass 0 -> 0.000001
- link prop2_link: mass 0 -> 0.000001
- link prop3_link: mass 0 -> 0.000001
Joints:
- joint prop0_joint: type fixed -> continuous
- joint prop1_joint: type fixed -> continuous
- joint prop2_joint: type fixed -> continuous
- joint prop3_joint: type fixed -> continuous
